File: Schematics/Circuit/main_polygon.kicad_pcb (KiCad board)
At the start: 2 copper layers, 59.3 x 59 mm, 93 parts, among them IC1 NCP1117ST33T3G, IC2 NCP1117ST50T3G, IC3 ATMEGA2560-A, IC4 RFM69HW, J1 Conn_01x03, J10 Conn_01x04, J2 Conn_01x07, J3 Conn_01x07, J4 Conn_01x07, J5 Conn_01x07, J6 Conn_01x07, J7 Conn_01x05, J8 Conn_02x05_Counter_Clockwise, J9 Conn_01x06, K1 HESOP1, K2 HESOP1, P1 CONN_2, P10 CONN_2, P11 CONN_2, P12 CONN_2, P13 CONN_2, P14 CONN_2, P15 CONN_2, P16 CONN_2, P17 CONN_2, P18 CONN_3X2, P19 CONN_O2, P2 CONN_2, P20 CONN_2, P21 CONN_2, P3 CONN_2, P4 CONN_2, P5 CONN_2, P6 CONN_2, P7 CONN_2, P8 CONN_2, P9 CONN_2, Q1 BSS138, Q2 BSS138, Q3 BSS138, Q4 BSS138, Q5 BSS138, Q6 BSS138

Commit message: Edit pcb and model
Parts:
- removed P11: CONN_2, CanSat:MOLEX_PicoBlade_2
- added J11: Conn_01x04, CanSat:MOLEX_PicoBlade_4, F.Cu at (56.1, 22.4)
- IC3: footprint ATMEGA2560-16AU:QFP50P1600X1600X120-100N -> CanSat:AtMega2560-AU
- P18: moved to F.Cu
- moved Q6 201.8 mm to (23.6, 59.1)
- moved R32 201.4 mm to (21.8, 60.9)
- moved R15 200.5 mm to (60.9, 33.7)
- moved IC4 200.4 mm to (41.1, 44.3)
- moved R24 200.3 mm to (52.7, 36.4)
- moved P18 200.2 mm to (55.3, 44.1)
- moved C1 200.2 mm to (30.5, 26.5)
- moved C10 200.2 mm to (32.5, 44.0)
- moved C11 200.2 mm to (38.3, 54.4)
- moved C12 200.2 mm to (47.7, 34.1)
- moved C13 200.2 mm to (35.6, 34.7)
- moved C14 200.2 mm to (54.5, 55.0)
- moved C2 200.2 mm to (37.5, 56.3)
- moved C6 200.2 mm to (40.1, 56.3)
- moved C7 200.2 mm to (43.9, 56.3)
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Connections:
- IC1 pad : (no net) -> +3V3
- IC3 pad 1: (no net) -> /INT2
- IC3 pad 12: (no net) -> /TXD-GSM
- IC3 pad 13: (no net) -> /RXD-GSM
- IC3 pad 14: (no net) -> /LED3
- IC3 pad 15: /PWM1 -> /PWM4
- IC3 pad 16: /PWM2 -> /PWM3
- IC3 pad 17: /PWM3 -> /PWM2
- IC3 pad 18: /PWM4 -> /PWM1
- IC3 pad 19: (no net) -> /INT3
- IC3 pad 24: (no net) -> /XSHUT3
- IC3 pad 27: (no net) -> Net-(IC3-Pad27)
- IC3 pad 28: /LED4 -> Net-(IC3-Pad28)
- IC3 pad 29: (no net) -> Net-(IC3-Pad29)
- IC3 pad 35: (no net) -> Net-(IC3-Pad35)
- IC3 pad 36: (no net) -> Net-(IC3-Pad36)
- IC3 pad 38: /PWM5 -> /PWM7
- IC3 pad 4: (no net) -> Net-(IC3-Pad4)
- IC3 pad 40: /PWM7 -> /PWM5
- IC3 pad 41: (no net) -> Net-(IC3-Pad41)
- IC3 pad 42: (no net) -> Net-(IC3-Pad42)
- IC3 pad 45: /TXD-GSM -> /INT1
- IC3 pad 46: /RXD-GSM -> Net-(IC3-Pad46)
- IC3 pad 48: /PWRKEY -> Net-(IC3-Pad48)
- IC3 pad 5: (no net) -> Net-(IC3-Pad5)
- IC3 pad 50: (no net) -> /XSHUT1
- IC3 pad 51: (no net) -> Net-(IC3-Pad51)
- IC3 pad 52: /LED2 -> Net-(IC3-Pad52)
- IC3 pad 53: /O2 -> Net-(IC3-Pad53)
- IC3 pad 54: /CO2 -> Net-(IC3-Pad54)
- IC3 pad 57: /LED_TOP -> Net-(IC3-Pad57)
- IC3 pad 58: (no net) -> Net-(IC3-Pad58)
- IC3 pad 59: (no net) -> /LED4
- IC3 pad 60: (no net) -> Net-(IC3-Pad60)
- IC3 pad 63: (no net) -> /RX_GPS
- IC3 pad 64: (no net) -> /TX_GPS
- IC3 pad 65: (no net) -> Net-(IC3-Pad65)
- IC3 pad 66: (no net) -> Net-(IC3-Pad66)
- IC3 pad 67: (no net) -> Net-(IC3-Pad67)
- IC3 pad 68: (no net) -> /INT4
- IC3 pad 69: (no net) -> Net-(IC3-Pad69)
- IC3 pad 70: /LED3 -> Net-(IC3-Pad70)
- IC3 pad 71: (no net) -> /XSHUT4
- IC3 pad 72: (no net) -> /LED_TOP
- IC3 pad 73: (no net) -> /PWRKEY
- IC3 pad 74: (no net) -> /SS
- IC3 pad 75: (no net) -> /CO2
- IC3 pad 76: (no net) -> /LED2
- IC3 pad 77: (no net) -> Net-(IC3-Pad77)
- IC3 pad 78: (no net) -> Net-(IC3-Pad78)
- IC3 pad 79: (no net) -> Net-(IC3-Pad79)
- IC3 pad 82: (no net) -> Net-(IC3-Pad82)
- IC3 pad 83: (no net) -> Net-(IC3-Pad83)
- IC3 pad 84: (no net) -> Net-(IC3-Pad84)
- IC3 pad 85: (no net) -> Net-(IC3-Pad85)
- IC3 pad 86: (no net) -> Net-(IC3-Pad86)
- IC3 pad 87: (no net) -> Net-(IC3-Pad87)
- IC3 pad 88: (no net) -> Net-(IC3-Pad88)
- IC3 pad 89: /SS -> Net-(IC3-Pad89)
- IC3 pad 90: (no net) -> Net-(IC3-Pad90)
- IC3 pad 91: (no net) -> Net-(IC3-Pad91)
- IC3 pad 92: (no net) -> Net-(IC3-Pad92)
- IC3 pad 93: (no net) -> Net-(IC3-Pad93)
- IC3 pad 94: /XSHUT4 -> Net-(IC3-Pad94)
- IC3 pad 95: /XSHUT3 -> Net-(IC3-Pad95)
- IC3 pad 97: /XSHUT1 -> /O2
- IC3 pad 98: (no net) -> Net-(IC3-Pad98)
- IC4 pad 1: (no net) -> Net-(IC4-Pad1)
- IC4 pad 10: (no net) -> Net-(IC4-Pad10)
- IC4 pad 16: (no net) -> Net-(IC4-Pad16)
- IC4 pad 3: (no net) -> Net-(IC4-Pad3)
- IC4 pad 4: (no net) -> Net-(IC4-Pad4)
- IC4 pad 5: (no net) -> Net-(IC4-Pad5)
- IC4 pad 6: (no net) -> Net-(IC4-Pad6)
- IC4 pad 7: (no net) -> Net-(IC4-Pad7)
- J10 pad : (no net) -> /CO2
- J2 pad : (no net) -> GND
- J3 pad : (no net) -> +5V
- J4 pad : (no net) -> /SCK
- J5 pad : (no net) -> /INT2
- J6 pad : (no net) -> /SDA
- J8 pad 1: (no net) -> /DTR
- J8 pad 6: (no net) -> Net-(J8-Pad6)
- J9 pad : (no net) -> /SCL
- K1 pad 3: (no net) -> Net-(K1-Pad3)
- K1 pad 4: (no net) -> Net-(K1-Pad4)
- K2 pad 3: (no net) -> Net-(K2-Pad3)
- K2 pad 4: (no net) -> Net-(K2-Pad4)
- P18 pad 4: (no net) -> Net-(P18-Pad4)
- P19 pad : (no net) -> GND
- P19 pad 3: (no net) -> Net-(P19-Pad3)
Routing:
- net +12V: track 226.9 -> 645.1 mm, vias 0 -> 3
- net GND: track 427.4 -> 792.4 mm, vias 13 -> 27
- net +5V: track 121.5 -> 311.9 mm, vias 9 -> 28
- net /SCL: track 33.3 -> 126.5 mm, vias 1 -> 10
- net +3V3: track 95.7 -> 177.6 mm, vias 7 -> 16
- net Net-(IC4-Pad14): track 2.78 -> 50.8 mm, vias 0 -> 7
- net /SDA: track 41.4 -> 89.0 mm, vias 2 -> 5
- net /RX: track 0.00 -> 43.4 mm, vias 0 -> 2
- net Net-(J2-Pad5): track 0.85 -> 42.6 mm, vias 0 -> 3
- net /RXD-GSM: track 0.00 -> 40.4 mm, vias 0 -> 5
- net /RX_GPS: track 0.00 -> 37.5 mm, vias 0 -> 2
- net /TX: track 0.00 -> 36.6 mm, vias 0 -> 2
- net /PWM8: track 0.00 -> 32.9 mm, vias 0 -> 2
- net /RFMINT: track 2.29 -> 33.0 mm, vias 0 -> 1
- net /TX_GPS: track 0.00 -> 30.4 mm, vias 0 -> 2
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Other:
- board size 59.3 x 59 mm -> 58.9 x 59 mm
- rule trace_min: 0.203 -> 0.197
