File: Schematics/Circuit/_autosave-main_polygon.kicad_pcb (KiCad board)
At the start: 2 copper layers, 58.9 x 59 mm, 93 parts, among them IC1 NCP1117ST33T3G, IC2 NCP1117ST50T3G, IC3 ATMEGA2560-A, IC4 RFM69HW, J1 Conn_01x03, J10 Conn_01x04, J11 Conn_01x04, J2 Conn_01x07, J3 Conn_01x07, J4 Conn_01x07, J5 Conn_01x07, J6 Conn_01x07, J7 Conn_01x05, J8 Conn_02x05_Counter_Clockwise, J9 Conn_01x06, K1 HESOP1, K2 HESOP1, P1 CONN_2, P10 CONN_2, P12 CONN_2, P13 CONN_2, P14 CONN_2, P15 CONN_2, P16 CONN_2, P17 CONN_2, P18 CONN_3X2, P19 CONN_O2, P2 CONN_2, P20 CONN_2, P21 CONN_2, P3 CONN_2, P4 CONN_2, P5 CONN_2, P6 CONN_2, P7 CONN_2, P8 CONN_2, P9 CONN_2, Q1 BSS138, Q2 BSS138, Q3 BSS138, Q4 BSS138, Q5 BSS138, Q6 BSS138

Commit message: Edit, add overall schematic, widen gaps in pcb
Routing:
- net GND: track 792.4 -> 796.0 mm
- net +3V3: track 177.6 -> 178.1 mm
Other:
- net class Default: clearance 0.197 -> 0.203
- rule trace_clearance: 0.197 -> 0.203
- rule trace_min: 0.197 -> 0.203
