File: CanSat2.0/Schematics/Circuit/center.kicad_pcb (KiCad board)
At the start: 2 copper layers, 23.9 x 86.5 mm, 35 parts, among them IC1 RFM69HW, J1 Main_connector, J10 SERVO_CONN, J11 FC_POWER, J12 GAMMA, J13 BOTTOM_CONN, J2 Conn_01x01, J3 FC_PWMS_A, J4 FC_PWMS_B, J5 Conn_01x07, J6 FC_OUTPUT, J7 DRIVERS_INPUT, J8 CAM_FM_CONN, J9 CAM_SD_CONN, Q1 BSS138, Q2 BSS138, Q3 Q_PMOS_GSD, Q4 Q_PMOS_GSD, Q6 BSS138

Commit message: Edit final version of pcbs, gerbers generated
Parts:
- removed R13, R5: 10k, Resistors_SMD:R_0805
- added REF**: Standoff, CanSat:Standoff, F.Cu at (38.2, 75.0)
- moved R6 7.49 mm to (41.6, 81.9)
- moved Q4 2.03 mm to (41.6, 79.2), turned to 90 degrees
- moved Q3 0.23 mm to (43.5, 50.0), turned to 180 degrees
Connections:
- J13 pad 4: +5V -> +3V3
- Q3 pad 2: /FC_PWR -> +5V
- Q3 pad 3: +5V -> /FC_PWR
- Q4 pad 2: /CAM_PWR -> +5V
- Q4 pad 3: +5V -> /CAM_PWR
Routing:
- net +5V: track 131.4 -> 116.6 mm, vias 4 -> 3
- net +3V3: track 112.7 -> 124.1 mm, vias 7 -> 8
- net /CAM_EN: track 54.4 -> 61.3 mm, vias 8 -> 10
- net /FC_EN: track 18.8 -> 21.6 mm
- net /SERVO: track 71.1 -> 73.4 mm
- net Net-(IC1-Pad2): track 51.4 -> 53.2 mm
- net /SDA: track 95.4 -> 96.8 mm
- net /GAMMA: track 62.7 -> 64.1 mm, vias 5 -> 3
- net Net-(IC1-Pad15): track 64.1 -> 63.4 mm, vias 6 -> 4
- net /FC_PWM_4: track 57.4 -> 56.7 mm
- net /FC_PWM_2: track 56.5 -> 57.1 mm
- net /FC_PWR: track 2.54 -> 3.06 mm
- net /MISOLOW: track 99.9 -> 99.8 mm, vias 4 -> 6
- net /SCKLOW: track 101.6 -> 101.7 mm, vias 10 -> 12
