File: CanSat2.0/Schematics/Circuit/center.sch (KiCad schematic (older format))
At the start: 32 parts

Commit message: Add three top boards and some other circuitry and modelling
Parts:
- removed J?: Center_connector, symbol Conn_02x11_Counter_Clockwise
- added J1: Main_connector, Pin_Headers:Pin_Header_Angled_2x13_Pitch1.27mm, symbol Conn_02x13_Odd_Even
- added J?: FC_OUTPUT, symbol Conn_01x04
- added J?: DRIVERS_INPUT, symbol Conn_01x04
- J3: renamed from J?; value Conn_01x04 -> FC_PWMS_A
- J4: renamed from J?; value Conn_01x04 -> FC_PWMS_B
- R1, R10, R11, R13, R14, R16, R18, R2, R3, R4, R5, R6, R7, R8, R9: renamed from R?; footprint Resistors_SMD:R_0603 -> Resistors_SMD:R_0805
- gave numbers to parts that had none: 14
Connections:
- net labels added: +3V3, MISOLOW, MOSILOW, MOT1, MOT2, MOT3, MOT4, SCKLOW, SCL, SDA, SERVO
- wire segments 90 -> 101
Other:
- moved on the sheet: IC1, J2, J3, J4, J5, Q1, Q2, Q3, Q4, Q5, Q6, R1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

Commit message: Add new pcbs - center and bottom - and fill the lower half of the model
Parts:
- removed Q3, Q4, Q5: BSS138, TO_SOT_Packages_SMD:SOT-23, symbol BSS138
- removed R10, R7, R8, R9: 10k, Resistors_SMD:R_0805, symbol R
- added J10: SERVO_CONN, Pin_Headers:Pin_Header_Straight_1x03_Pitch2.54mm, symbol Conn_01x03
- added J11: FC_POWER, Pin_Headers:Pin_Header_Straight_1x02_Pitch2.54mm, symbol Conn_01x02
- added J12: GAMMA, Pin_Headers:Pin_Header_Straight_1x04_Pitch2.54mm, symbol Conn_01x04
- added J13: BOTTOM_CONN, Pin_Headers:Pin_Header_Angled_1x04_Pitch2.54mm, symbol Conn_01x04
- added J8: CAM_FM_CONN, Pin_Headers:Pin_Header_Straight_1x02_Pitch2.54mm, symbol Conn_01x02
- added J9: CAM_SD_CONN, Pin_Headers:Pin_Header_Straight_1x04_Pitch2.54mm, symbol Conn_01x04
- added Q3, Q4: Q_PMOS_GSD, TO_SOT_Packages_SMD:SOT-23, symbol Q_PMOS_GSD
- IC1: footprint RFM69HW:XCVR_RFM95W-868S2 -> CanSat:RFM69HW
- J3, J4: footprint (none) -> Pin_Headers:Pin_Header_Straight_1x04_Pitch1.27mm
- J5: footprint CanSat:MOLEX_PicoBlade_7 -> Pin_Headers:Pin_Header_Straight_1x07_Pitch2.54mm
- J6: renamed from J?; footprint (none) -> Pin_Headers:Pin_Header_Straight_1x04_Pitch2.54mm
- J7: renamed from J?; footprint (none) -> Pin_Headers:Pin_Header_Straight_1x05_Pitch1.27mm; symbol Conn_01x04 -> Conn_01x05
- R20: footprint Resistors_SMD:R_0603 -> Resistors_SMD:R_0805
Connections:
- net labels added: CAM_PWR, FC_PWR, GAMMA
- net labels removed: MISO, MOSI, PWRKEY, RXD-GSM, SCK, SLEEP-GSM, TXD-GSM
- wire segments 101 -> 130
Other:
- moved on the sheet: J2, J6, Q2, R3, R5

Commit message: Edit final version of pcbs, gerbers generated
Parts:
- removed R13, R5: 10k, Resistors_SMD:R_0805, symbol R
Other:
- moved on the sheet: Q4, R14, R6
