File: CanSat2.0/Schematics/Circuit/main.sch (KiCad schematic (older format))
At the start: 38 parts, among them J1 Center connector, J2 Middle connector, P1 CONN_2, P15 CONN_2, P2 CONN_2, P3 CONN_2, P4 CONN_2, SW7 SW_DIP_x01, U1 LD1117S33TR_SOT223, U2 O2, U3 LD1117S50TR_SOT223, U4 mg812_gas_sensor, U5 AD8572, U6 SP3_gas_sensor, U7 LMC662

Commit message: PCBs
Parts:
- added SW?: SW_DIP_x01, symbol SW_DIP_x01
Connections:
- wire segments 163 -> 164
Changed lines of the file:
@@
 L +BATT #PWR03
 U 1 1 5AE2A246
-P 1400 5100
-F 0 "#PWR03" H 1400 4950 50  0001 C CNN
-F 1 "+BATT" H 1400 5240 50  0000 C CNN
-F 2 "" H 1400 5100 50  0001 C CNN
-F 3 "" H 1400 5100 50  0001 C CNN
-	1    1400 5100
+P 1400 4200
+F 0 "#PWR03" H 1400 4050 50  0001 C CNN
+F 1 "+BATT" H 1400 4340 50  0000 C CNN
+F 2 "" H 1400 4200 50  0001 C CNN
+F 3 "" H 1400 4200 50  0001 C CNN
+	1    1400 4200
 	1    0    0    -1
 $EndComp
@@
 Connection ~ 1400 6850
 Wire Wire Line
-	1400 5100 1400 5650
+	1400 4200 1400 4750
 Wire Wire Line
 	1400 5650 1450 5650
@@
 Text Label 8800 2750 0    60   ~ 0
 SDA
+$Comp
+L SW_DIP_x01 SW?
+U 1 1 5AF42AEC
+P 1400 5050
+F 0 "SW?" H 1400 5200 50  0000 C CNN
+F 1 "SW_DIP_x01" H 1400 4900 50  0000 C CNN
+F 2 "" H 1400 5050 50  0001 C CNN
+F 3 "" H 1400 5050 50  0001 C CNN
+	1    1400 5050
+	0    -1   -1   0
+$EndComp
+Wire Wire Line
+	1400 5350 1400 5650
 $EndSCHEMATC

Commit message: Add three top boards and some other circuitry and modelling
Parts:
- removed J2: Middle connector, Pin_Headers:Pin_Header_Straight_2x15_Pitch1.27mm, symbol Conn_02x15_Counter_Clockwise
- added J2: Conn_02x08_Counter_Clockwise, Pin_Headers:Pin_Header_Straight_2x08_Pitch1.27mm, symbol Conn_02x08_Odd_Even
- added J3: Conn_02x07_Counter_Clockwise, Pin_Headers:Pin_Header_Straight_2x07_Pitch1.27mm, symbol Conn_02x07_Odd_Even
- J1: symbol Conn_02x13_Counter_Clockwise -> Conn_02x13_Odd_Even
- SW1: renamed from SW?; footprint (none) -> CanSat:TX30_vertical
Connections:
- net labels added: MISOLOW, MOSILOW, SCKLOW
- net labels removed: MISO, MOSI, SCK
Other:
- moved on the sheet: C1, C14, C2, C3, C4, C5, C6, C7, C8, C9, P1, P15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

Commit message: Add new pcbs - center and bottom - and fill the lower half of the model
Parts:
- J3: symbol Conn_02x07_Odd_Even -> Conn_02x07_Counter_Clockwise
Connections:
- net labels added: GAMMA
- wire segments 164 -> 166

Commit message: Edit final version of pcbs, gerbers generated
Parts:
- added C10, C11: 100 nF, Capacitors_SMD:C_0805, symbol C-RESCUE-main
- added unit 2 of U7
Connections:
- wire segments 166 -> 180
Other:
- moved on the sheet: P4
Changed lines of the file:
@@
 L CONN_2 P4
 U 1 1 5AE8CD76
-P 8100 5850
-F 0 "P4" V 8050 5850 40  0000 C CNN
-F 1 "CONN_2" V 8150 5850 40  0000 C CNN
-F 2 "CanSat:TX30_vertical" H 8100 5850 60  0001 C CNN
-F 3 "" H 8100 5850 60  0000 C CNN
-	1    8100 5850
+P 8900 5850
+F 0 "P4" V 8850 5850 40  0000 C CNN
+F 1 "CONN_2" V 8950 5850 40  0000 C CNN
+F 2 "CanSat:TX30_vertical" H 8900 5850 60  0001 C CNN
+F 3 "" H 8900 5850 60  0000 C CNN
+	1    8900 5850
 	1    0    0    -1
 $EndComp
@@
 L +BATT #PWR017
 U 1 1 5AE8CF14
-P 7650 5650
-F 0 "#PWR017" H 7650 5500 50  0001 C CNN
-F 1 "+BATT" H 7650 5790 50  0000 C CNN
-F 2 "" H 7650 5650 50  0001 C CNN
-F 3 "" H 7650 5650 50  0001 C CNN
-	1    7650 5650
+P 8450 5650
+F 0 "#PWR017" H 8450 5500 50  0001 C CNN
+F 1 "+BATT" H 8450 5790 50  0000 C CNN
+F 2 "" H 8450 5650 50  0001 C CNN
+F 3 "" H 8450 5650 50  0001 C CNN
+	1    8450 5650
 	1    0    0    -1
 $EndComp
@@
 L GND #PWR022
 U 1 1 5AE8DC31
-P 7650 6050
-F 0 "#PWR022" H 7650 5800 50  0001 C CNN
-F 1 "GND" H 7650 5900 50  0000 C CNN
-F 2 "" H 7650 6050 50  0001 C CNN
-F 3 "" H 7650 6050 50  0001 C CNN
-	1    7650 6050
+P 8450 6050
+F 0 "#PWR022" H 8450 5800 50  0001 C CNN
+F 1 "GND" H 8450 5900 50  0000 C CNN
+F 2 "" H 8450 6050 50  0001 C CNN
+F 3 "" H 8450 6050 50  0001 C CNN
+	1    8450 6050
 	1    0    0    -1
 $EndComp
@@
 	1650 5650 1650 5350
 Connection ~ 1050 5350
-Connection ~ 1050 6100
-Connection ~ 1650 6100
 Wire Wire Line
 	950  1350 950  2150
@@
 	1750 2500 1750 2450
 Wire Wire Line
-	3650 4850 5600 4850
+	3650 4850 6200 4850
 Wire Wire Line
 	3750 4850 3750 4750
@@
 Connection ~ 4550 3800
 Wire Wire Line
-	5300 4050 5400 4050
+	5300 4050 6200 4050
 Wire Wire Line
 	5400 4050 5400 4000
@@
 	7600 1550 7700 1550
 Wire Wire Line
-	7650 5650 7650 5750
-Wire Wire Line
-	7650 5750 7750 5750
-Wire Wire Line
-	7750 5950 7650 5950
-Wire Wire Line
-	7650 5950 7650 6050
+	8450 5650 8450 5750
+Wire Wire Line
+	8450 5750 8550 5750
+Wire Wire Line
+	8550 5950 8450 5950
+Wire Wire Line
+	8450 5950 8450 6050
 Wire Wire Line
 	1650 6850 1050 6850
@@
 Text Label 8600 5050 2    60   ~ 0
 GAMMA
+Wire Wire Line
+	5300 4450 5350 4450
+Wire Wire Line
+	5350 4450 5350 4850
+Connection ~ 5350 4850
+Wire Wire Line
+	5300 4550 5350 4550
+Connection ~ 5350 4550
+$Comp
+L LMC6482 U7
+U 2 1 5B111423
+P 7000 6000
+F 0 "U7" H 7000 6200 50  0000 L CNN
+F 1 "LMC662" H 7000 5800 50  0000 L CNN
+F 2 "Housings_SOIC:SOIC-8_3.9x4.9mm_Pitch1.27mm" H 7000 6000 50  0001 C CNN
+F 3 "" H 7000 6000 50  0001 C CNN
+	2    7000 6000
+	1    0    0    -1
+$EndComp
+$Comp
+L GND #PWR028
+U 1 1 5B11151E
+P 6600 6500
+F 0 "#PWR028" H 6600 6250 50  0001 C CNN
+F 1 "GND" H 6600 6350 50  0000 C CNN
+F 2 "" H 6600 6500 50  0001 C CNN
+F 3 "" H 6600 6500 50  0001 C CNN
+	1    6600 6500
+	1    0    0    -1
+$EndComp
+Wire Wire Line
+	6900 6300 6900 6400
+Wire Wire Line
+	6600 6400 7550 6400
+Wire Wire Line
+	6600 5900 6600 6500
+Wire Wire Line
+	6700 6100 6600 6100
+Connection ~ 6600 6400
+Wire Wire Line
+	6700 5900 6600 5900
+Connection ~ 6600 6100
+$Comp
+L +5V #PWR029
+U 1 1 5B111834
+P 6900 5600
+F 0 "#PWR029" H 6900 5450 50  0001 C CNN
+F 1 "+5V" H 6900 5740 50  0000 C CNN
+F 2 "" H 6900 5600 50  0001 C CNN
+F 3 "" H 6900 5600 50  0001 C CNN
+	1    6900 5600
+	1    0    0    -1
+$EndComp
+Wire Wire Line
+	6900 5600 6900 5700
+$Comp
+L C-RESCUE-main C10
+U 1 1 5B113FFE
+P 6200 4350
+F 0 "C10" H 6200 4450 40  0000 L CNN
+F 1 "100 nF" H 6206 4265 40  0000 L CNN
+F 2 "Capacitors_SMD:C_0805" H 6238 4200 30  0000 C CNN
+F 3 "~" H 6200 4350 60  0000 C CNN
+	1    6200 4350
+	1    0    0    -1
+$EndComp
+Wire Wire Line
+	6200 4050 6200 4150
+Connection ~ 5400 4050
+Wire Wire Line
+	6200 4850 6200 4550
+$Comp
+L C-RESCUE-main C11
+U 1 1 5B114589
+P 7550 6000
+F 0 "C11" H 7550 6100 40  0000 L CNN
+F 1 "100 nF" H 7556 5915 40  0000 L CNN
+F 2 "Capacitors_SMD:C_0805" H 7588 5850 30  0000 C CNN
+F 3 "~" H 7550 6000 60  0000 C CNN
+	1    7550 6000
+	1    0    0    -1
+$EndComp
+Wire Wire Line
+	6900 5650 7550 5650
+Wire Wire Line
+	7550 5650 7550 5800
+Connection ~ 6900 5650
+Wire Wire Line
+	7550 6400 7550 6200
+Connection ~ 6900 6400
 $EndSCHEMATC
