File: CanSat2.0/Schematics/Circuit/middle.kicad_pcb (KiCad board)
At the start: 2 copper layers, 64 x 64 mm, 34 parts, among them IC1 ATMEGA2560-A, J1 Conn_02x05_Counter_Clockwise, J2 Conn_02x08_Counter_Clockwise, J3 Conn_01x08, J4 Conn_02x07_Counter_Clockwise, J5 Conn_01x04, Q1 BSS138, Q2 BSS138, Q3 BSS138, Q4 BSS138, U1 SD

Commit message: Edit final version of pcbs, gerbers generated
Parts:
- removed R11, R6, R7, R8: 10k, Resistors_SMD:R_0805
- added C8: 10 uF, Capacitors_Tantalum_SMD:CP_Tantalum_Case-B_EIA-3528-21_Reflow, F.Cu at (50.1, 65.3)
- added C9: 10 uF, Capacitors_Tantalum_SMD:CP_Tantalum_Case-B_EIA-3528-21_Reflow, F.Cu at (30.9, 58.2)
- added L1: 10 uH, Inductors_SMD:L_Taiyo-Yuden_NR-50xx, F.Cu at (33.1, 53.5)
- added L2: Ferrite_Bead, Inductors_SMD:L_0805, B.Cu at (41.6, 57.4)
- moved C7 0.63 mm to (35.0, 58.4), turned to 270 degrees
Connections:
- C4 pad 1: +5V -> Net-(C4-Pad1)
- C5 pad 1: +5V -> Net-(C4-Pad1)
- C6 pad 1: +5V -> Net-(C4-Pad1)
- C7 pad 1: +5V -> GND
- C7 pad 2: GND -> Net-(C7-Pad2)
- IC1 pad 10: +5V -> Net-(C4-Pad1)
- IC1 pad 100: +5V -> Net-(C7-Pad2)
- IC1 pad 16: /FC_PWM_3 -> (no net)
- IC1 pad 17: /FC_PWM_2 -> (no net)
- IC1 pad 31: +5V -> Net-(C4-Pad1)
- IC1 pad 43: /SDA -> /SCL
- IC1 pad 44: /SCL -> /SDA
- IC1 pad 45: /RX_GPS -> /TX_GPS
- IC1 pad 46: /TX_GPS -> /RX_GPS
- IC1 pad 76: (no net) -> /FC_PWM_2
- IC1 pad 77: (no net) -> /FC_PWM_3
- IC1 pad 80: +5V -> Net-(C4-Pad1)
- J2 pad 10: /FC_PWM_7 -> /FC_PWM_5
- J2 pad 11: /FC_PWM_6 -> /GSM_SLP
- J2 pad 12: /FC_PWM_5 -> /FC_PWM_6
- J2 pad 13: /FC_PWM_4 -> /GSM_KEY
- J2 pad 14: /FC_PWM_3 -> /FC_PWM_7
- J2 pad 15: /FC_PWM_2 -> /GSM_TX
- J2 pad 16: /FC_PWM_1 -> /FC_PWM_8
- J2 pad 2: +3V3 -> /FC_PWM_1
- J2 pad 3: GND -> +3V3
- J2 pad 4: /CAM_EN -> /FC_PWM_2
- J2 pad 5: /FC_EN -> GND
- J2 pad 6: /GSM_SLP -> /FC_PWM_3
- J2 pad 7: /GSM_KEY -> /CAM_EN
- J2 pad 8: /GSM_TX -> /FC_PWM_4
- J2 pad 9: /FC_PWM_8 -> /FC_EN
Routing:
- net Net-(C4-Pad1): track 0.00 -> 52.5 mm, vias 0 -> 8
- net /FC_PWM_3: track 53.8 -> 19.5 mm, vias 4 -> 2
- net /FC_PWM_4: track 27.0 -> 54.0 mm, vias 3 -> 4
- net /FC_PWM_6: track 23.6 -> 47.5 mm, vias 3 -> 4
- net /GSM_TX: track 48.2 -> 27.6 mm, vias 2 -> 3
- net /FC_PWM_8: track 29.0 -> 48.4 mm, vias 5 -> 7
- net +5V: track 156.9 -> 140.0 mm, vias 7 -> 9
- net GND: track 141.9 -> 158.0 mm, vias 13 -> 9
- net /GSM_SLP: track 20.5 -> 6.48 mm, vias 2 -> 1
- net /CAM_EN: track 18.0 -> 7.48 mm, vias 2 -> 0
- net Net-(C7-Pad2): track 0.00 -> 9.66 mm, vias 0 -> 1
- net /FC_PWM_2: track 25.7 -> 16.2 mm, vias 3 -> 2
- net /FC_PWM_1: track 26.6 -> 33.8 mm, vias 3 -> 4
- net /FC_PWM_7: track 44.2 -> 49.5 mm
- net /MOSILOW: track 47.4 -> 52.5 mm, vias 5 -> 3
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Other:
- outline, holes or cut-outs redrawn
- net class Default: clearance 0.165 -> 0.164
- rule trace_clearance: 0.165 -> 0.164
