File: CanSat2.0/Schematics/Circuit/middle.sch (KiCad schematic (older format))
At the start: 16 parts, among them IC1 ATMEGA2560-A, J1 Conn_02x05_Counter_Clockwise, J2 Main connector, J3 Conn_01x09

Commit message: Add three top boards and some other circuitry and modelling
Parts:
- removed J2: Main connector, Pin_Headers:Pin_Header_Straight_2x15_Pitch1.27mm, symbol Conn_02x15_Counter_Clockwise
- added J2: Conn_02x08_Counter_Clockwise, Pin_Headers:Pin_Header_Straight_2x08_Pitch1.27mm, symbol Conn_02x08_Counter_Clockwise
- added J4: Conn_02x07_Counter_Clockwise, Pin_Headers:Pin_Header_Straight_2x08_Pitch1.27mm, symbol Conn_02x07_Counter_Clockwise
- added J5: Conn_01x04, Pin_Headers:Pin_Header_Straight_1x04_Pitch1.27mm, symbol Conn_01x04
- added Q1, Q2, Q3, Q4: BSS138, TO_SOT_Packages_SMD:SOT-23, symbol BSS138
- added R10, R11, R12, R5, R6, R7, R8, R9: 10k, Resistors_SMD:R_0603, symbol R
- added U1: SD, CanSat:SD, symbol SD
- J3: value Conn_01x09 -> Conn_01x08; footprint Pin_Headers:Pin_Header_Straight_1x09_Pitch1.27mm -> Pin_Headers:Pin_Header_Straight_1x08_Pitch1.27mm; symbol Conn_01x09 -> Conn_01x08
Connections:
- net labels added: LED1, LED2, LED3, LED4, MISOLOW, MOSILOW, SCKLOW, SD_SS, SD_SSLOW
- net labels removed: CAM_TRIG, DTR, FLY_TRIG, GSM_SLEEP, LED, LED_TOP, RXD-GSM, SS, TXD-GSM
- wire segments 114 -> 143
Other:
- moved on the sheet: C1, C2, C3, C4, C5, C6, C7, CSTECE1, IC1, J1, R1, R2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

Commit message: Add new pcbs - center and bottom - and fill the lower half of the model
Parts:
- J4: footprint Pin_Headers:Pin_Header_Straight_2x08_Pitch1.27mm -> Pin_Headers:Pin_Header_Straight_2x07_Pitch1.27mm
- R10, R11, R12, R5, R6, R7, R8, R9: footprint Resistors_SMD:R_0603 -> Resistors_SMD:R_0805
Connections:
- net labels added: GAMMA
- net labels removed: INT4
- wire segments 143 -> 144
Changed lines of the file:
@@
 Text Label 5950 2000 0    60   ~ 0
 GSM_KEY
-Text Label 3100 4600 0    60   ~ 0
-INT4
 Text Label 6000 3000 0    60   ~ 0
 SERVO
@@
 	5900 2000 6300 2000
 Wire Wire Line
-	3100 4600 3300 4600
-Wire Wire Line
 	5900 3000 6300 3000
 Wire Wire Line
@@
 Wire Wire Line
 	1750 1900 1750 1800
-Text Label 10150 950  0    60   ~ 0
+Text Label 10600 950  2    60   ~ 0
 FC_PWM_1
-Text Label 10150 1050 0    60   ~ 0
+Text Label 10600 1050 2    60   ~ 0
 FC_PWM_2
-Text Label 10150 1150 0    60   ~ 0
+Text Label 10600 1150 2    60   ~ 0
 FC_PWM_3
-Text Label 10150 1250 0    60   ~ 0
+Text Label 10600 1250 2    60   ~ 0
 FC_PWM_4
-Text Label 10150 1350 0    60   ~ 0
+Text Label 10600 1350 2    60   ~ 0
 FC_PWM_5
-Text Label 10150 1450 0    60   ~ 0
+Text Label 10600 1450 2    60   ~ 0
 FC_PWM_6
-Text Label 10150 1550 0    60   ~ 0
+Text Label 10600 1550 2    60   ~ 0
 FC_PWM_7
-Text Label 10150 1650 0    60   ~ 0
+Text Label 10600 1650 2    60   ~ 0
 FC_PWM_8
 $Comp
@@
 $EndComp
 Wire Wire Line
-	10150 950  10550 950
-Wire Wire Line
-	10150 1050 10550 1050
-Wire Wire Line
-	10150 1150 10550 1150
-Wire Wire Line
-	10150 1250 10550 1250
-Wire Wire Line
-	10150 1350 10550 1350
-Wire Wire Line
-	10150 1450 10550 1450
-Wire Wire Line
-	10150 1550 10550 1550
-Wire Wire Line
-	10150 1650 10550 1650
+	10150 950  10600 950
+Wire Wire Line
+	10150 1050 10600 1050
+Wire Wire Line
+	10150 1150 10600 1150
+Wire Wire Line
+	10150 1250 10600 1250
+Wire Wire Line
+	10150 1350 10600 1350
+Wire Wire Line
+	10150 1450 10600 1450
+Wire Wire Line
+	10150 1550 10600 1550
+Wire Wire Line
+	10150 1650 10600 1650
 Wire Wire Line
 	10150 2200 10550 2200
@@
 Wire Wire Line
 	9550 950  9650 950
-Text Label 10250 2200 0    60   ~ 0
+Text Label 10550 2200 2    60   ~ 0
 RFM_INT
-Text Label 10250 2300 0    60   ~ 0
+Text Label 10550 2300 2    60   ~ 0
 RFM_SS
-Text Label 10200 2400 0    60   ~ 0
+Text Label 10550 2400 2    60   ~ 0
 MOSILOW
 Text Label 9250 2400 0    60   ~ 0
@@
 Text Label 9250 2600 0    60   ~ 0
 CO2
-Text Label 10450 2500 0    60   ~ 0
+Text Label 10550 2500 2    60   ~ 0
 O3
-Text Label 10250 2600 0    60   ~ 0
+Text Label 10550 2600 2    60   ~ 0
 V_READ
 $Comp
@@
 	1    0    0    -1
 $EndComp
-Text Label 10300 2700 0    60   ~ 0
+Text Label 10550 2700 2    60   ~ 0
 SERVO
 Wire Wire Line
@@
 Wire Wire Line
 	3150 3700 3300 3700
-Wire Wire Line
-	9250 2700 9650 2700
-Wire Wire Line
-	9650 2800 9250 2800
-Text Label 9250 2700 0    60   ~ 0
-SCL
-Text Label 9250 2800 0    60   ~ 0
-SDA
 $Comp
 L GND #PWR013
@@
 F 0 "J4" H 9900 2900 50  0000 C CNN
 F 1 "Conn_02x07_Counter_Clockwise" H 9900 2100 50  0000 C CNN
-F 2 "Pin_Headers:Pin_Header_Straight_2x08_Pitch1.27mm" H 9850 2500 50  0001 C CNN
+F 2 "Pin_Headers:Pin_Header_Straight_2x07_Pitch1.27mm" H 9850 2500 50  0001 C CNN
 F 3 "" H 9850 2500 50  0001 C CNN
 	1    9850 2500
@@
 F 0 "R5" V 8130 3900 50  0000 C CNN
 F 1 "10k" V 8050 3900 50  0000 C CNN
-F 2 "Resistors_SMD:R_0603" V 7980 3900 50  0001 C CNN
+F 2 "Resistors_SMD:R_0805" V 7980 3900 50  0001 C CNN
 F 3 "" H 8050 3900 50  0001 C CNN
 	1    8050 3900
@@
 F 0 "R8" V 8630 3900 50  0000 C CNN
 F 1 "10k" V 8550 3900 50  0000 C CNN
-F 2 "Resistors_SMD:R_0603" V 8480 3900 50  0001 C CNN
+F 2 "Resistors_SMD:R_0805" V 8480 3900 50  0001 C CNN
 F 3 "" H 8550 3900 50  0001 C CNN
 	1    8550 3900
@@
 F 0 "R6" V 8130 4900 50  0000 C CNN
 F 1 "10k" V 8050 4900 50  0000 C CNN
-F 2 "Resistors_SMD:R_0603" V 7980 4900 50  0001 C CNN
+F 2 "Resistors_SMD:R_0805" V 7980 4900 50  0001 C CNN
 F 3 "" H 8050 4900 50  0001 C CNN
 	1    8050 4900
@@
 F 0 "R9" V 8630 4900 50  0000 C CNN
 F 1 "10k" V 8550 4900 50  0000 C CNN
-F 2 "Resistors_SMD:R_0603" V 8480 4900 50  0001 C CNN
+F 2 "Resistors_SMD:R_0805" V 8480 4900 50  0001 C CNN
 F 3 "" H 8550 4900 50  0001 C CNN
 	1    8550 4900
@@
 F 0 "R7" V 8130 5800 50  0000 C CNN
 F 1 "10k" V 8050 5800 50  0000 C CNN
-F 2 "Resistors_SMD:R_0603" V 7980 5800 50  0001 C CNN
+F 2 "Resistors_SMD:R_0805" V 7980 5800 50  0001 C CNN
 F 3 "" H 8050 5800 50  0001 C CNN
 	1    8050 5800
@@
 F 0 "R10" V 8630 5800 50  0000 C CNN
 F 1 "10k" V 8550 5800 50  0000 C CNN
-F 2 "Resistors_SMD:R_0603" V 8480 5800 50  0001 C CNN
+F 2 "Resistors_SMD:R_0805" V 8480 5800 50  0001 C CNN
 F 3 "" H 8550 5800 50  0001 C CNN
 	1    8550 5800
@@
 F 0 "R11" V 9730 3900 50  0000 C CNN
 F 1 "10k" V 9650 3900 50  0000 C CNN
-F 2 "Resistors_SMD:R_0603" V 9580 3900 50  0001 C CNN
+F 2 "Resistors_SMD:R_0805" V 9580 3900 50  0001 C CNN
 F 3 "" H 9650 3900 50  0001 C CNN
 	1    9650 3900
@@
 F 0 "R12" V 10230 3900 50  0000 C CNN
 F 1 "10k" V 10150 3900 50  0000 C CNN
-F 2 "Resistors_SMD:R_0603" V 10080 3900 50  0001 C CNN
+F 2 "Resistors_SMD:R_0805" V 10080 3900 50  0001 C CNN
 F 3 "" H 10150 3900 50  0001 C CNN
 	1    10150 3900
@@
 Wire Wire Line
 	6900 1100 7150 1100
+Text Label 6000 5500 0    60   ~ 0
+GAMMA
+Wire Wire Line
+	6300 5500 5900 5500
+Wire Wire Line
+	10550 2800 10150 2800
+Text Label 10550 2800 2    60   ~ 0
+GAMMA
+Text Label 9250 2700 0    60   ~ 0
+SCL
+Text Label 9250 2800 0    60   ~ 0
+SDA
+Wire Wire Line
+	9650 2700 9250 2700
+Wire Wire Line
+	9650 2800 9250 2800
 $EndSCHEMATC

Commit message: Edit final version of pcbs, gerbers generated
Parts:
- removed R11, R6, R7, R8: 10k, Resistors_SMD:R_0805, symbol R
- added C8, C9: 10 uF, Capacitors_Tantalum_SMD:CP_Tantalum_Case-B_EIA-3528-21_Reflow, symbol CP1
- added L1: 10 uH, Inductors_SMD:L_Taiyo-Yuden_NR-50xx, symbol L
- added L2: Ferrite_Bead, Inductors_SMD:L_0805, symbol Ferrite_Bead
- J2: symbol Conn_02x08_Counter_Clockwise -> Conn_02x08_Odd_Even
Connections:
- wire segments 144 -> 167
Other:
- moved on the sheet: C1, C2, C3, C4, C5, C6, C7, CSTECE1, IC1, J1, R1, R2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
