File: CanSat2.0/Schematics/Circuit/top.sch (KiCad schematic (older format))
At the start: 29 parts, among them J1 Conn_01x09, K1 SI7021, Q1 BSS138, Q2 BSS138, U1 LSM303AGRTR, U2 VEML6070, U3 TSL2591, U4 microservo, U5 GPS, U6 MPL3115A2

Commit message: Add three top boards and some other circuitry and modelling
Parts:
- added D2, D3, D4: LED, Diodes_SMD:D_0603, symbol LED-RESCUE-top
- added J2: Conn_01x04, Pin_Headers:Pin_Header_Straight_1x04_Pitch1.27mm, symbol Conn_01x04
- added R10, R8, R9: 105, Resistors_SMD:R_0805, symbol R
- J1: value Conn_01x09 -> Conn_01x08; footprint Pin_Headers:Pin_Header_Straight_1x09_Pitch1.27mm_SMD_Pin1Left -> Pin_Headers:Pin_Header_Straight_1x08_Pitch1.27mm; symbol Conn_01x09 -> Conn_01x08
- R1: value 150 -> 105
- U5: footprint (none) -> CanSat:GPS
Connections:
- net labels added: LED1, LED2, LED3, LED4
- net labels removed: LED
- wire segments 105 -> 122
Other:
- moved on the sheet: D1, R1

Commit message: Edit final version of pcbs, gerbers generated
Parts:
- removed R5, R6: 10k, Resistors_SMD:R_0805, symbol R
- added C12: 10 uF, Capacitors_Tantalum_SMD:CP_Tantalum_Case-T_EIA-3528-12_Reflow, symbol CP1
Connections:
- wire segments 122 -> 123
Changed lines of the file:
@@
 LED1
 $Comp
-L +3.3V #PWR26
+L +3.3V #PWR25
 U 1 1 5A5BAF55
 P 9800 3800
-F 0 "#PWR26" H 9800 3650 50  0001 C CNN
+F 0 "#PWR25" H 9800 3650 50  0001 C CNN
 F 1 "+3.3V" H 9800 3940 50  0000 C CNN
 F 2 "" H 9800 3800 50  0001 C CNN
@@
 SCL
 $Comp
-L GND #PWR22
+L GND #PWR23
 U 1 1 5AE09854
 P 8700 1600
-F 0 "#PWR22" H 8700 1350 50  0001 C CNN
+F 0 "#PWR23" H 8700 1350 50  0001 C CNN
 F 1 "GND" H 8700 1450 50  0000 C CNN
 F 2 "" H 8700 1600 50  0001 C CNN
@@
 $EndComp
 $Comp
-L +3V3 #PWR29
+L +3V3 #PWR28
 U 1 1 5AE0987C
 P 10350 1000
-F 0 "#PWR29" H 10350 850 50  0001 C CNN
+F 0 "#PWR28" H 10350 850 50  0001 C CNN
 F 1 "+3V3" H 10350 1140 50  0000 C CNN
 F 2 "" H 10350 1000 50  0001 C CNN
@@
 F 3 "" H 8450 6000 50  0001 L CNN
 	1    8450 6000
-	0    1    1    0
+	0    -1   1    0
 $EndComp
 $Comp
@@
 	-1   0    0    1
 $EndComp
-$Comp
-L R R5
-U 1 1 5AE21403
-P 8750 5850
-F 0 "R5" V 8830 5850 50  0000 C CNN
-F 1 "10k" V 8750 5850 50  0000 C CNN
-F 2 "Resistors_SMD:R_0805" V 8680 5850 50  0001 C CNN
-F 3 "" H 8750 5850 50  0001 C CNN
-	1    8750 5850
-	-1   0    0    1
-$EndComp
 Text Label 8800 6100 0    60   ~ 0
 TX_GPSL
@@
 	7600 4400 7600 4300
 Wire Wire Line
-	4200 5700 3750 5700
+	3550 5700 4200 5700
 Wire Wire Line
 	3750 5700 3750 5600
 Wire Wire Line
-	4200 5800 3750 5800
+	3550 5800 4200 5800
 Wire Wire Line
 	3750 5800 3750 5900
@@
 	8650 6100 9150 6100
 Wire Wire Line
-	8750 6000 8750 6100
-Connection ~ 8750 6100
-Wire Wire Line
-	8750 5500 8750 5700
-Wire Wire Line
-	8750 5600 8450 5600
-Wire Wire Line
-	8450 5600 8450 5800
+	8450 5500 8450 5800
 Wire Wire Line
 	8150 5700 8150 5500
-Connection ~ 8750 5600
-$Comp
-L +3V3 #PWR23
+$Comp
+L +3V3 #PWR22
 U 1 1 5AE21A7F
-P 8750 5500
-F 0 "#PWR23" H 8750 5350 50  0001 C CNN
-F 1 "+3V3" H 8750 5640 50  0000 C CNN
-F 2 "" H 8750 5500 50  0001 C CNN
-F 3 "" H 8750 5500 50  0001 C CNN
-	1    8750 5500
+P 8450 5500
+F 0 "#PWR22" H 8450 5350 50  0001 C CNN
+F 1 "+3V3" H 8450 5640 50  0000 C CNN
+F 2 "" H 8450 5500 50  0001 C CNN
+F 3 "" H 8450 5500 50  0001 C CNN
+	1    8450 5500
 	1    0    0    -1
 $EndComp
@@
 F 3 "" H 10050 6000 50  0001 L CNN
 	1    10050 6000
-	0    1    1    0
-$EndComp
-$Comp
-L R R6
-U 1 1 5AE21C29
-P 9750 5850
-F 0 "R6" V 9830 5850 50  0000 C CNN
-F 1 "10k" V 9750 5850 50  0000 C CNN
-F 2 "Resistors_SMD:R_0805" V 9680 5850 50  0001 C CNN
-F 3 "" H 9750 5850 50  0001 C CNN
-	1    9750 5850
-	-1   0    0    1
+	0    -1   1    0
 $EndComp
 $Comp
@@
 	9350 6100 9850 6100
 Wire Wire Line
-	9750 6000 9750 6100
-Connection ~ 9750 6100
-Wire Wire Line
 	10250 6100 10750 6100
 Wire Wire Line
@@
 Wire Wire Line
 	10050 5600 10050 5800
-Wire Wire Line
-	9750 5700 9750 5500
 Connection ~ 10350 5600
 $Comp
-L +3V3 #PWR30
+L +3V3 #PWR29
 U 1 1 5AE21C42
 P 10350 5500
-F 0 "#PWR30" H 10350 5350 50  0001 C CNN
+F 0 "#PWR29" H 10350 5350 50  0001 C CNN
 F 1 "+3V3" H 10350 5640 50  0000 C CNN
 F 2 "" H 10350 5500 50  0001 C CNN
 F 3 "" H 10350 5500 50  0001 C CNN
 	1    10350 5500
-	1    0    0    -1
-$EndComp
-$Comp
-L +5V #PWR25
-U 1 1 5AE21C48
-P 9750 5500
-F 0 "#PWR25" H 9750 5350 50  0001 C CNN
-F 1 "+5V" H 9750 5640 50  0000 C CNN
-F 2 "" H 9750 5500 50  0001 C CNN
-F 3 "" H 9750 5500 50  0001 C CNN
-	1    9750 5500
 	1    0    0    -1
 $EndComp
@@
 	10750 4200 10700 4200
 $Comp
-L +3V3 #PWR27
+L +3V3 #PWR26
 U 1 1 5B054ADA
 P 10200 1900
-F 0 "#PWR27" H 10200 1750 50  0001 C CNN
+F 0 "#PWR26" H 10200 1750 50  0001 C CNN
 F 1 "+3V3" H 10200 2040 50  0000 C CNN
 F 2 "" H 10200 1900 50  0001 C CNN
@@
 $EndComp
 $Comp
-L GND #PWR28
+L GND #PWR27
 U 1 1 5B054AFD
 P 10200 2700
-F 0 "#PWR28" H 10200 2450 50  0001 C CNN
+F 0 "#PWR27" H 10200 2450 50  0001 C CNN
 F 1 "GND" H 10200 2550 50  0000 C CNN
 F 2 "" H 10200 2700 50  0001 C CNN
@@
 Wire Wire Line
 	5200 2450 5200 2550
+$Comp
+L CP1 C12
+U 1 1 5B11731F
+P 3250 5750
+F 0 "C12" H 3275 5850 50  0000 L CNN
+F 1 "10 uF" H 3275 5650 50  0000 L CNN
+F 2 "Capacitors_Tantalum_SMD:CP_Tantalum_Case-T_EIA-3528-12_Reflow" H 3250 5750 50  0001 C CNN
+F 3 "" H 3250 5750 50  0001 C CNN
+	1    3250 5750
+	1    0    0    -1
+$EndComp
+Wire Wire Line
+	3250 5600 3250 5500
+Wire Wire Line
+	3250 5500 3550 5500
+Wire Wire Line
+	3550 5500 3550 5700
+Connection ~ 3750 5700
+Wire Wire Line
+	3550 5800 3550 6000
+Wire Wire Line
+	3550 6000 3250 6000
+Wire Wire Line
+	3250 6000 3250 5900
+Connection ~ 3750 5800
 $EndSCHEMATC
